Commit message: adding links for wheels

File: src/robot_description/urdf/auto_vehicle.urdf.xacro (robot description, xacro)
@@ -101,9 +101,85 @@
         </inertial>
     </link>
-    <!-- Wheels Using Macro -->
-    <xacro:wheel name="left_back_wheel"/>
-    <xacro:wheel name="right_back_wheel"/>
-    <xacro:wheel name="left_front_wheel"/>
-    <xacro:wheel name="right_front_wheel"/>
+    <!-- Wheels as Links -->
+    <link name="left_back_wheel">
+        <visual>
+            <geometry>
+                <cylinder radius="${wheel_radius}" length="${wheel_length}"/>
+            </geometry>
+            <origin xyz="0 0 0" rpy="0 1.57 0"/>
+            <material name="black"/>
+        </visual>
+        <collision>
+            <geometry>
+                <cylinder radius="${wheel_radius}" length="${wheel_length}"/>
+            </geometry>
+            <origin xyz="0 0 0" rpy="0 1.57 0"/>
+        </collision>
+        <inertial>
+            <mass value="0.5"/>
+            <origin xyz="0 0 0" rpy="0 0 0"/>
+            <inertia ixx="0.0016" ixy="0.0" ixz="0.0" iyy="0.000867" iyz="0.0" izz="0.000867"/>
+        </inertial>
+    </link>
+    <link name="right_back_wheel">
+        <visual>
+            <geometry>
+                <cylinder radius="${wheel_radius}" length="${wheel_length}"/>
+            </geometry>
+            <origin xyz="0 0 0" rpy="0 1.57 0"/>
+            <material name="black"/>
+        </visual>
+        <collision>
+            <geometry>
+                <cylinder radius="${wheel_radius}" length="${wheel_length}"/>
+            </geometry>
+            <origin xyz="0 0 0" rpy="0 1.57 0"/>
+        </collision>
+        <inertial>
+            <mass value="0.5"/>
+            <origin xyz="0 0 0" rpy="0 0 0"/>
+            <inertia ixx="0.0016" ixy="0.0" ixz="0.0" iyy="0.000867" iyz="0.0" izz="0.000867"/>
+        </inertial>
+    </link>
+    <link name="left_front_wheel">
+        <visual>
+            <geometry>
+                <cylinder radius="${wheel_radius}" length="${wheel_length}"/>
+            </geometry>
+            <origin xyz="0 0 0" rpy="0 1.57 0"/>
+            <material name="black"/>
+        </visual>
+        <collision>
+            <geometry>
+                <cylinder radius="${wheel_radius}" length="${wheel_length}"/>
+            </geometry>
+            <origin xyz="0 0 0" rpy="0 1.57 0"/>
+        </collision>
+        <inertial>
+            <mass value="0.5"/>
+            <origin xyz="0 0 0" rpy="0 0 0"/>
+            <inertia ixx="0.0016" ixy="0.0" ixz="0.0" iyy="0.000867" iyz="0.0" izz="0.000867"/>
+        </inertial>
+    </link>
+    <link name="right_front_wheel">
+        <visual>
+            <geometry>
+                <cylinder radius="${wheel_radius}" length="${wheel_length}"/>
+            </geometry>
+            <origin xyz="0 0 0" rpy="0 1.57 0"/>
+            <material name="black"/>
+        </visual>
+        <collision>
+            <geometry>
+                <cylinder radius="${wheel_radius}" length="${wheel_length}"/>
+            </geometry>
+            <origin xyz="0 0 0" rpy="0 1.57 0"/>
+        </collision>
+        <inertial>
+            <mass value="0.5"/>
+            <origin xyz="0 0 0" rpy="0 0 0"/>
+            <inertia ixx="0.0016" ixy="0.0" ixz="0.0" iyy="0.000867" iyz="0.0" izz="0.000867"/>
+        </inertial>
+    </link>
     <!-- Joints -->
     <xacro:fixed_joint
